File: hardware/product/Product-Programmable/EsperDNS.sch (KiCad schematic (older format))
At the start: 0 parts

Commit message: Updated schematic to be more readable
Parts:
- added C1, C12, C4, C9: 1uF, Capacitor_SMD:C_0402_1005Metric, symbol Device:C
- added C10, C3: 10uF, Capacitor_SMD:C_0805_2012Metric, symbol Device:C
- added C11, C2, C5, C6, C7, C8: 0.1uF, Capacitor_SMD:C_0402_1005Metric, symbol Device:C
- added D1: GRN, Diode_SMD:D_0603_1608Metric, symbol Device:LED
- added D2: RS-3535MWAR, LED_SMD:LED_RGB_PLCC-6, symbol LED:ASMT-YTB7-0AA02
- added FB2: Ferrite_Bead, Inductor_SMD:L_0805_2012Metric, symbol Device:Ferrite_Bead
- added H1, H2: MountingHole, MountingHole:MountingHole_2.2mm_M2_Pad, symbol Mechanical:MountingHole_Pad
- added J1: USB_B_Micro, Connector_USB:USB_Micro-B_Molex-105017-0001, symbol Connector:USB_B_Micro
- added J3: RJ45_Amphenol_RJMG1BD3B8K1ANR, Connector_RJ:RJ45_Amphenol_RJMG1BD3B8K1ANR, symbol Connector:RJ45_Amphenol_RJMG1BD3B8K1ANR
- added Q1, Q2, Q3, Q4, Q5: 2N7002, Package_TO_SOT_SMD:SOT-23, symbol Device:Q_NMOS_GSD
- added R1: 470, Resistor_SMD:R_0402_1005Metric, symbol Device:R
- added R10, R11, R12, R2, R24, R8: 10K, Resistor_SMD:R_0402_1005Metric, symbol Device:R
- added R13, R14, R15, R16, R18, R19, R20, R22, R6, R7, R9: 49.9, Resistor_SMD:R_0402_1005Metric, symbol Device:R
- added R17, R21: 270, Resistor_SMD:R_0603_1608Metric, symbol Device:R
- added R23: 12.1K, Resistor_SMD:R_0402_1005Metric, symbol Device:R
- added R3, R4: 47, Resistor_SMD:R_0603_1608Metric, symbol Device:R
- added R5: 82, Resistor_SMD:R_1206_3216Metric, symbol Device:R
- added SW1: PTS645VH83-2 LFS, Button_Switch_THT:SW_Tactile_SPST_Angled_PTS645Vx83-2LFS, symbol Switch:SW_SPST
- added U1: AZ1117EH-3.3TRG1, Package_TO_SOT_SMD:SOT-223, symbol Regulator_Linear:AZ1117-3.3
- added U2: ESP32-WROOM-32E, RF_Module:ESP32-WROOM-32, symbol RF_Module:ESP32-WROOM-32D
- added U3: LAN8720A, Package_DFN_QFN:QFN-24-1EP_4x4mm_P0.5mm_EP2.6x2.6mm_ThermalVias, symbol Interface_Ethernet:LAN8720A
- added U4: CP2102-GMR_NRND, EsperFootprints:VFQFN-28-1EP_5x5mm, symbol EsperSymbols:CP2102-GMR_NRND
Connections:
- new net: Q3.3 (D), R3.2
- new net: Q2.3 (D), R4.2
- new net: Q1.3 (D), R5.2
- new net: D2.2 (KG), R4.1
- new net: D2.1 (KB), R3.1
- new net: D2.3 (KR), R5.1
- new net: D1.2 (A), R1.2
- new net +3.3VA: C10.1, C11.1, C4.1, C5.1, C6.1, FB2.1, J3.R4 (TCT), J3.R5 (RCT), R10.1, R11.1, R12.1, R13.1, R14.1, R15.1, R16.1, R17.1, U3.1 (VDD2A), U3.19 (VDD1A)
- new net +3V3: C3.1, C7.1, FB2.2, R1.1, R2.2, U1.2 (VO), U2.2 (VDD), U3.9 (VDDIO), U4.6 (VDD)
- new net Block: R8.2, SW1.2 (B), U2.6 (IO34)
- new net Blue: Q3.1 (G), U2.27 (IO16)
- new net CLK50MHZ: R22.1, U3.5 (XTAL1/CLKIN)
- new net CLK_R: R22.2, U2.28 (IO17)
- new net CRS_DV: R20.2, U2.12 (IO27)
- new net CRS_DV_R: R20.1, U3.11 (CRS_DV/MODE2)
- new net D+: J1.3 (D+), U4.4 (D+)
- new net D-: J1.2 (D-), U4.5 (D-)
- new net DTR: Q4.2 (S), Q5.1 (G), U4.28 (DTR)
- new net EN: C12.1, Q5.3 (D), R2.1, U2.3 (EN)
- new net Earth: H1.1, H2.1, J1.6 (Shield), J3.13 (SHIELD)
- new net GND: C1.2, C10.2, C11.2, C12.2, C2.2, C3.2, C4.2, C5.2, C6.2, C7.2, C8.2, C9.2, D1.1 (K), J1.5 (GND), J3.R8 (GND), Q1.2 (S), Q2.2 (S), Q3.2 (S), R21.2, R23.2, R24.2, SW1.1 (A), U1.1 (GND), U2.1 (GND), U2.15 (GND), U2.38 (GND), U2.39 (GND), U3.25 (VSS), U4.29 (GND_PAD), U4.3 (GND)
- new net Green: Q2.1 (G), U2.9 (IO33)
- new net IO0: Q4.3 (D), U2.25 (IO0)
- new net LED1_REGOFF: J3.L4 (LEDG_A), U3.3 (LED1/REGOFF)
- new net LED2_nINTSEL: J3.L2 (LEDY_K), U3.2 (LED2/nINTSEL)
- new net LEDG_K: J3.L3 (LEDG_K), R21.1
- new net LEDY_A: J3.L1 (LEDY_A), R17.2
- new net MDC: U2.37 (IO23), U3.13 (MDC)
- new net MDIO: R10.2, U2.30 (IO18), U3.12 (MDIO)
- new net MTCK: U2.16 (IO13)
- new net MTDI: U2.14 (IO12)
- new net MTDO: U2.23 (IO15)
- new net MTMS: U2.13 (IO14)
- new net PHYAD0: R24.1, U3.10 (RXER/PHYAD0)
- new net RBIAS: R23.1, U3.24 (RBIAS)
- new net RD+: J3.R3 (RD+), R15.2, U3.23 (RXP)
- new net RD-: J3.R6 (RD-), R16.2, U3.22 (RXN)
- new net RTS: Q4.1 (G), Q5.2 (S), U4.24 (RTS)
- new net RX: U2.35 (TXD0/IO1), U4.25 (RXD)
- new net RX0_R: R18.1, U3.8 (RXD0/MODE0)
- new net RX1_R: R19.1, U3.7 (RXD1/MODE1)
- new net RXD0: R18.2, U2.10 (IO25)
- new net RXD1: R19.2, U2.11 (IO26)
- new net Red: Q1.1 (G), U2.8 (IO32)
- new net TD+: J3.R1 (TD+), R13.2, U3.21 (TXP)
- new net TD-: J3.R2 (TD-), R14.2, U3.20 (TXN)
- new net TX: U2.34 (RXD0/IO3), U4.26 (TXD)
- new net TXD0: R6.2, U3.17 (TXD0)
- new net TXD0_R: R6.1, U2.31 (IO19)
- new net TXD1: R9.2, U3.18 (TXD1)
- new net TXD1_R: R9.1, U2.36 (IO22)
- new net TXEN: R7.2, U3.16 (TXEN)
- new net TXEN_R: R7.1, U2.33 (IO21)
- new net VBUS: C1.1, C2.1, D2.4 (AR), D2.5 (AG), D2.6 (AB), J1.1 (VBUS), R8.1, U1.3 (VI), U4.7 (REGIN), U4.8 (VBUS), U4.9 (RST)
- new net VDDCR: C8.1, C9.1, U3.6 (VDDCR)
- new net nINT: R12.2, U2.7 (IO35), U3.14 (INT/REFCLKO)
- new net nRST: R11.2, U2.26 (IO4), U3.15 (RST)
- no-connect marks 0 -> 34
Other:
- note added: "5V Vbus to 3.3V"
- note added: "Auto program\nDTR RTS-->EN IO0\n 1 1 1 1\n 0 0 1 1\n 1 0 0 1\n 0 1 1 0"
- note added: "Automatically puts ESP32 in programming mode when using ESP-IDF.\n\nhttps://github.com/espressif/esptool/wiki/ESP32-Boot-Mode-Selection#automatic-bootloader"
- note added: "Button & LEDs"
- note added: "Can't use for LEDs, \nPulled up during startup:\n1, 3, 6, 7, 8, \n9, 10, 11, 14"
- note added: "Decoupling Caps, place near U2"
- note added: "ESP32"
- note added: "Ethernet"
- note added: "Input Only:\n34, 35, SENSOR_VP, SENSOR_VN"
- note added: "MODE[2:0] have internal pull-ups\nCurrently configured for:\n-10/100BASE\n-Auto-negoation enabled\n-SMI address = 0x00\n-nINT enabled, REFCLKO disabled\n-VDDCR enabled"
- note added: "Need 1uF for \ncircuit to work"
- note added: "No decoupling needed\n10uf, 1uf, 0.1uf caps inside\n"
- note added: "Programming"
- note added: "RED: 2.2V @ 40mA\nGREEN: 3.5V @ 40mA\nBLUE: 3.5V @ 40mA\n"
- note added: "Strapping Pins:\n• GPIO0: internal pull-up\n• GPIO2: internal pull-down\n• GPIO4: internal pull-down\n• GPIO5: internal pull-up\n• MTDI/GPIO12: internal pull-down\n• MTDO/GPIO15: internal pull-up"
